Commit message: move_base_to_goal(predefined poses) move_base_to_pose(with x,y,yaw input) move_arm_cartesian_position_component(ik for arm)

File: edufill_sw/edufill_common/edufill_robot_description/urdf/sensors/asus_xtion_camera.urdf.xacro (robot description, xacro)
@@ -28,5 +28,5 @@
         <origin xyz="0.01 0 0" rpy="${M_PI/2} 0 ${M_PI/2}" />
         <geometry>
-           <mesh filename="package://raw_robot_description/meshes/sensors/asus_xtion_pro_live_base.dae" scale="0.0004 0.0007 0.001"/>
+           <mesh filename="package://edufill_robot_description/meshes/sensors/asus_xtion_pro_live_base.dae" scale="0.0004 0.0007 0.001"/>
         </geometry>
         <material name="Black" />
@@ -35,5 +35,5 @@
         <origin xyz="0.01 0 0" rpy="${M_PI/2} 0 ${M_PI/2}" />
         <geometry>
-           <mesh filename="package://raw_robot_description/meshes/sensors/asus_xtion_pro_live_base.dae" scale="0.0004 0.0007 0.001"/>
+           <mesh filename="package://edufill_robot_description/meshes/sensors/asus_xtion_pro_live_base.dae" scale="0.0004 0.0007 0.001"/>
         </geometry>
       </collision >
@@ -81,5 +81,5 @@
         <origin xyz="0.02 -0.03 0" rpy="${M_PI/2} 0 ${M_PI/2}" />
         <geometry>
-          <mesh filename="package://raw_robot_description/meshes/sensors/asus_xtion_pro_live_camera.dae" scale="0.001 0.001 0.001"/>
+          <mesh filename="package://edufill_robot_description/meshes/sensors/asus_xtion_pro_live_camera.dae" scale="0.001 0.001 0.001"/>
         </geometry>
         <material name="Black" />
@@ -88,5 +88,5 @@
         <origin xyz="0.02 -0.03 0" rpy="${M_PI/2} 0 ${M_PI/2}" />
         <geometry>
-           <mesh filename="package://raw_robot_description/meshes/sensors/asus_xtion_pro_live_camera.dae" scale="0.001 0.001 0.001"/>
+           <mesh filename="package://edufill_robot_description/meshes/sensors/asus_xtion_pro_live_camera.dae" scale="0.001 0.001 0.001"/>
         </geometry>
       </collision >

File: edufill_sw/edufill_common/edufill_robot_description/urdf/sensors/kinect_camera.urdf.xacro (robot description, xacro)
@@ -22,5 +22,5 @@
       <origin xyz="0.0 0.0 0.0" rpy="0 0 0" />
       <geometry>
-       <mesh filename="package://raw_robot_description/meshes/sensors/kinect.dae"/>
+       <mesh filename="package://edufill_robot_description/meshes/sensors/kinect.dae"/>
       </geometry>
     </visual>
@@ -28,5 +28,5 @@
       <origin xyz="0.0 0.0 0.0" rpy="0 0 0" />
       <geometry>
-        <mesh filename="package://raw_robot_description/meshes/sensors/kinect.dae"/>
+        <mesh filename="package://edufill_robot_description/meshes/sensors/kinect.dae"/>
       </geometry>
     </collision>

File: edufill_sw/edufill_common/edufill_robot_description/urdf/sensors/microsoft_lifecam.urdf.xacro (robot description, xacro)
@@ -22,5 +22,5 @@
       <origin xyz="-0.04 -0.0035 -0.031" rpy="${M_PI/2} 0 ${M_PI/2}" />
       <geometry>
-       <mesh filename="package://raw_robot_description/meshes/sensors/microsoft_lifecam.dae" scale="0.001 0.001 0.001"/>
+       <mesh filename="package://edufill_robot_description/meshes/sensors/microsoft_lifecam.dae" scale="0.001 0.001 0.001"/>
       </geometry>
     </visual>
@@ -28,5 +28,5 @@
       <origin xyz="-0.04 -0.0035 -0.031" rpy="${M_PI/2} 0 ${M_PI/2}" />
       <geometry>
-        <mesh filename="package://raw_robot_description/meshes/sensors/microsoft_lifecam.dae" scale="0.001 0.001 0.001"/>
+        <mesh filename="package://edufill_robot_description/meshes/sensors/microsoft_lifecam.dae" scale="0.001 0.001 0.001"/>
       </geometry>
     </collision>
