Commit message: changes to afford simulation in fuerte!!!

File: edufill_sw/edufill_robots/edufill_robot_config/edufill_hardware_config/youbot-edufill2/urdf/youbot-edufill2.urdf.xacro (robot description, xacro)
@@ -41,9 +41,9 @@
   <!-- BRSU SPECIFIC STUFF -->
   <include filename="$(find edufill_robot_description)/urdf/materials.urdf.xacro" />
-  <!--include filename="$(find raw_robot_description)/urdf/misc/sensor_angle.urdf.xacro" /-->
+  <!--include filename="$(find edufill_robot_description)/urdf/misc/sensor_angle.urdf.xacro" /-->
   <include filename="$(find edufill_robot_description)/urdf/misc/cam3d_tower.urdf.xacro" />
   <include filename="$(find edufill_robot_description)/urdf/sensors/kinect_camera.urdf.xacro" />
-  <!--include filename="$(find raw_robot_description)/urdf/sensors/microsoft_lifecam.urdf.xacro" /-->
-  <!--include filename="$(find raw_robot_description)/urdf/sensors/asus_xtion_camera.urdf.xacro" /-->
+  <!--include filename="$(find edufill_robot_description)/urdf/sensors/microsoft_lifecam.urdf.xacro" /-->
+  <!--include filename="$(find edufill_robot_description)/urdf/sensors/asus_xtion_camera.urdf.xacro" /-->
   <!-- base laser rear -->
   <xacro:hokuyo_urg04_laser name="base_laser_rear" parent="base" ros_topic="scan_rear" update_rate="10" min_angle="-1.57" max_angle="1.57" >
@@ -63,6 +63,6 @@
   </xacro:cam3d_tower>
   <!-- 3D camera on tower -->
-  <xacro:kinect_camera name="openni" parent="tower_link">
-    <origin xyz="0.0509 -0.03 0.49" rpy="0 0.545 0" />
+  <xacro:kinect_camera name="tower_cam3d" parent="tower_link">
+    <origin xyz="0.0509 -0.03 0.49" rpy="0.0 0.545 0.0" />
   </xacro:kinect_camera>
   <!-- Microsoft LifeCam on gripper -->

File: edufill_sw/edufill_simulation/edufill_gazebo_world/common/worlds/brsu-home.urdf.xacro (robot description, xacro)
@@ -11,5 +11,5 @@
 									Wall 3
 -->
-<robot name="arena">
+<robot name="brsu-c025-arena">
   	<link name="wall_1">
     		<inertial>
@@ -297,49 +297,49 @@
   <gazebo reference="wall_1">
 	<material>Gazebo/White</material>
-	<selfCollide>true</selfCollide>
+	<selfCollide>false</selfCollide>
   </gazebo>
   <gazebo reference="wall_2">
 	<material>Gazebo/White</material>
-	<selfCollide>true</selfCollide>
+	<selfCollide>false</selfCollide>
   </gazebo>
   <gazebo reference="wall_3">
 	<material>Gazebo/White</material>
-	<selfCollide>true</selfCollide>
+	<selfCollide>false</selfCollide>
   </gazebo>
   <gazebo reference="wall_4">
 	<material>Gazebo/White</material>
-	<selfCollide>true</selfCollide>
+	<selfCollide>false</selfCollide>
   </gazebo>
   <gazebo reference="wall_5">
 	<material>Gazebo/White</material>
-	<selfCollide>true</selfCollide>
+	<selfCollide>false</selfCollide>
   </gazebo>
   <gazebo reference="wall_6">
 	<material>Gazebo/White</material>
-	<selfCollide>true</selfCollide>
+	<selfCollide>false</selfCollide>
   </gazebo>
   <gazebo reference="wall_7">
 	<material>Gazebo/White</material>
-	<selfCollide>true</selfCollide>
+	<selfCollide>false</selfCollide>
   </gazebo>
   <gazebo reference="wall_8">
 	<material>Gazebo/White</material>
-	<selfCollide>true</selfCollide>
+	<selfCollide>false</selfCollide>
   </gazebo>
   <gazebo reference="wall_9">
 	<material>Gazebo/White</material>
-	<selfCollide>true</selfCollide>
+	<selfCollide>false</selfCollide>
   </gazebo>
   <gazebo reference="wall_10">
 	<material>Gazebo/White</material>
-	<selfCollide>true</selfCollide>
+	<selfCollide>false</selfCollide>
   </gazebo>
   <gazebo reference="wall_11">
 	<material>Gazebo/White</material>
-	<selfCollide>true</selfCollide>
+	<selfCollide>false</selfCollide>
   </gazebo>
   <gazebo reference="wall_12">
 	<material>Gazebo/White</material>
-	<selfCollide>true</selfCollide>
+	<selfCollide>false</selfCollide>
   </gazebo>
 </robot>
